File: KiCAD/RCM-Hardware-D1/RCM-Hardware-D1.kicad_sch (KiCad schematic)
At the start: 2 parts, among them U1 WeMos_D1_mini, U2 L293D

Commit message: Continued the KeyCAD for the circuit board
Parts:
- added C1: C_Polarized, Capacitor_THT:C_Radial_D8.0mm_H11.5mm_P3.50mm, symbol Device:C_Polarized
- added J1, J2: Conn_01x02_Pin, Connector_PinSocket_2.54mm:PinSocket_1x02_P2.54mm_Vertical, symbol Connector:Conn_01x02_Pin
- added J3: battery, project:battery wires, symbol Connector:Conn_01x02_Pin
- added J6: Conn_01x04_Pin, Connector_JST:JST_SH_SM04B-SRSS-TB_1x04-1MP_P1.00mm_Horizontal, symbol Connector:Conn_01x04_Pin
- added J7: Conn_01x06_Pin, Connector_PinHeader_2.54mm:PinHeader_2x03_P2.54mm_Vertical, symbol Connector:Conn_01x06_Pin
- added R1, R2: R, Resistor_THT:R_Axial_DIN0204_L3.6mm_D1.6mm_P5.08mm_Horizontal, symbol Device:R
Connections:
- net GND: now also C1.2, J3.2 (Pin_2), J6.1 (Pin_1), J7.1 (Pin_1), J7.2 (Pin_2), R2.1
- net at U1.13 (D2): now also J6.3 (Pin_3), J7.5 (Pin_5)
- net at U1.14 (D1): now also J6.4 (Pin_4), J7.6 (Pin_6)
- net at U1.2 (A0): now also R1.1, R2.2
- net at U1.3 (D0): now also U2.7 (2A)
- net at U1.4 (D5): now also U2.10 (3A)
- net at U1.5 (D6): now also U2.15 (4A)
- net at U1.6 (D7): now also U2.2 (1A)
- net +3.3V: now reaches U1.8 (3.3V)
- net +3.3V: now also U2.1 (EN1,2), U2.9 (EN3,4), J6.2 (Pin_2)
- net at U1.9 (5V): now also U2.16 (VCC1), U2.8 (VCC2), C1.1, J3.1 (Pin_1), J7.3 (Pin_3), J7.4 (Pin_4), R1.2
- net at U2.11 (3Y): now also J1.2 (Pin_2)
- net at U2.14 (4Y): now also J1.1 (Pin_1)
- net at U2.3 (1Y): now also J2.2 (Pin_2)
- net at U2.6 (2Y): now also J2.1 (Pin_1)

Commit message: finished the KiCAD and created Gerbers
Connections:
- net GND: now also C1.1, J3.1 (Pin_1), J7.3 (Pin_3), J7.4 (Pin_4), R1.2, U1.9 (5V), U2.16 (VCC1), U2.8 (VCC2)
Other:
- moved on the sheet: U1
Changed lines of the file:
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@@
+	)
+	(junction
+		(at 118.11 74.93)
+		(diameter 0)
+		(color 0 0 0 0)
 	)
 	(junction
@@
 	)
 	(junction
+		(at 118.11 66.04)
+		(diameter 0)
+		(color 0 0 0 0)
+	)
+	(junction
 		(at 120.65 83.82)
 		(diameter 0)
@@
 	)
 	(junction
-		(at 120.65 74.93)
-		(diameter 0)
-		(color 0 0 0 0)
-	)
-	(junction
 		(at 153.67 102.87)
 		(diameter 0)
@@
 	(wire
 		(pts
-			(xy 81.28 68.58) (xy 95.25 68.58)
-		)
-		(stroke
-			(width 0)
-			(type default)
-		)
-	)
-	(wire
-		(pts
-			(xy 120.65 66.04) (xy 124.46 66.04)
-		)
-		(stroke
-			(width 0)
-			(type default)
-		)
-	)
-	(wire
-		(pts
-			(xy 120.65 55.88) (xy 152.4 55.88)
+			(xy 88.9 66.04) (xy 92.71 66.04)
+		)
+		(stroke
+			(width 0)
+			(type default)
+		)
+	)
+	(wire
+		(pts
+			(xy 118.11 53.34) (xy 152.4 53.34)
 		)
 		(stroke
@@
 	(wire
 		(pts
-			(xy 152.4 55.88) (xy 152.4 71.12)
+			(xy 88.9 68.58) (xy 81.28 68.58)
+		)
+		(stroke
+			(width 0)
+			(type default)
+		)
+	)
+	(wire
+		(pts
+			(xy 152.4 53.34) (xy 152.4 71.12)
 		)
 		(stroke
@@
 	(wire
 		(pts
-			(xy 81.28 45.72) (xy 81.28 53.34)
+			(xy 81.28 45.72) (xy 81.28 50.8)
 		)
 		(stroke
@@
 	(wire
 		(pts
-			(xy 68.58 55.88) (xy 68.58 102.87)
+			(xy 68.58 53.34) (xy 68.58 102.87)
 		)
 		(stroke
@@
 	(wire
 		(pts
-			(xy 120.65 58.42) (xy 128.27 58.42)
+			(xy 118.11 55.88) (xy 128.27 55.88)
 		)
 		(stroke
@@
 	(wire
 		(pts
-			(xy 95.25 55.88) (xy 68.58 55.88)
+			(xy 92.71 53.34) (xy 68.58 53.34)
 		)
 		(stroke
@@
 	(wire
 		(pts
-			(xy 95.25 63.5) (xy 71.12 63.5)
+			(xy 92.71 60.96) (xy 71.12 60.96)
 		)
 		(stroke
@@
 	(wire
 		(pts
-			(xy 77.47 58.42) (xy 95.25 58.42)
+			(xy 77.47 55.88) (xy 92.71 55.88)
 		)
 		(stroke
@@
 	(wire
 		(pts
+			(xy 118.11 66.04) (xy 124.46 66.04)
+		)
+		(stroke
+			(width 0)
+			(type default)
+		)
+	)
+	(wire
+		(pts
 			(xy 120.65 118.11) (xy 128.27 118.11)
 		)
@@
 	(wire
 		(pts
-			(xy 120.65 74.93) (xy 120.65 68.58)
+			(xy 118.11 74.93) (xy 118.11 66.04)
 		)
 		(stroke
@@
 	(wire
 		(pts
-			(xy 97.79 74.93) (xy 120.65 74.93)
+			(xy 97.79 74.93) (xy 118.11 74.93)
 		)
 		(stroke
@@
 	(wire
 		(pts
-			(xy 71.12 63.5) (xy 71.12 97.79)
-		)
-		(stroke
-			(width 0)
-			(type default)
-		)
-	)
-	(wire
-		(pts
-			(xy 73.66 60.96) (xy 95.25 60.96)
+			(xy 71.12 60.96) (xy 71.12 97.79)
+		)
+		(stroke
+			(width 0)
+			(type default)
+		)
+	)
+	(wire
+		(pts
+			(xy 88.9 66.04) (xy 88.9 68.58)
+		)
+		(stroke
+			(width 0)
+			(type default)
+		)
+	)
+	(wire
+		(pts
+			(xy 73.66 58.42) (xy 92.71 58.42)
 		)
 		(stroke
@@
 	(wire
 		(pts
-			(xy 73.66 60.96) (xy 73.66 118.11)
+			(xy 73.66 58.42) (xy 73.66 118.11)
 		)
 		(stroke
@@
 	(wire
 		(pts
+			(xy 118.11 63.5) (xy 118.11 66.04)
+		)
+		(stroke
+			(width 0)
+			(type default)
+		)
+	)
+	(wire
+		(pts
 			(xy 153.67 102.87) (xy 153.67 106.68)
 		)
@@
 	(wire
 		(pts
-			(xy 81.28 53.34) (xy 95.25 53.34)
-		)
-		(stroke
-			(width 0)
-			(type default)
-		)
-	)
-	(wire
-		(pts
-			(xy 128.27 58.42) (xy 128.27 73.66)
+			(xy 81.28 50.8) (xy 92.71 50.8)
+		)
+		(stroke
+			(width 0)
+			(type default)
+		)
+	)
+	(wire
+		(pts
+			(xy 128.27 55.88) (xy 128.27 73.66)
 		)
 		(stroke
@@
 	(wire
 		(pts
-			(xy 77.47 58.42) (xy 77.47 113.03)
+			(xy 118.11 74.93) (xy 120.65 74.93)
+		)
+		(stroke
+			(width 0)
+			(type default)
+		)
+	)
+	(wire
+		(pts
+			(xy 77.47 55.88) (xy 77.47 113.03)
 		)
 		(stroke
@@
 	(symbol
 		(lib_id "projlib:WeMos_D1_mini")
-		(at 107.95 59.69 0)
+		(at 105.41 57.15 0)
 		(unit 1)
 		(exclude_from_sim no)
@@
 		(dnp no)
 		(property "Reference" "U1"
-			(at 107.95 41.148 0)
+			(at 105.41 38.608 0)
 			(effects
 				(font
@@
 		)
 		(property "Value" "WeMos_D1_mini"
-			(at 107.95 43.18 0)
+			(at 105.41 40.64 0)
 			(effects
 				(font
@@
 		)
 		(property "Footprint" "project:wemos-d1-mini-with-pin-header"
-			(at 107.95 43.18 0)
+			(at 105.41 40.64 0)
 			(effects
 				(font
@@
 		)
 		(property "Datasheet" "http://www.wemos.cc/Products/d1_mini.html"
-			(at 107.95 45.72 0)
+			(at 105.41 43.18 0)
 			(effects
 				(font
@@
 		)
 		(property "Description" "WeMos D1 mini"
-			(at 107.95 59.69 0)
-			(effects
-				(font
+			(at 105.41 57.15 0)
+			(effects
+				(font
