File: KiCAD/RCM-Hardware-D1/RCM-Hardware-D1.kicad_pcb (KiCad board)
At the start: 2 copper layers, 33 x 55.9 mm, 2 parts, among them U1 WeMos_D1_mini, U2 L293D

Commit message: set up kicad
Parts:
- U2: moved to F.Cu
- moved U2 20.9 mm to (134.6, 76.2), turned to 0 degrees
Other:
- board size 33 x 55.9 mm -> 66 x 63.5 mm

Commit message: update kicad
Parts:
- moved U2 19.1 mm to (115.6, 77.5)
Connections:
- U1 pad 10: unconnected-(U1-GND-Pad10) -> GND
- U2 pad 12: unconnected-(U2-GND-Pad12) -> GND
- U2 pad 13: unconnected-(U2-GND-Pad13) -> GND
- U2 pad 4: unconnected-(U2-GND-Pad4) -> GND
- U2 pad 5: unconnected-(U2-GND-Pad5) -> GND
Changed lines of the file:
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@@
 		(0 "F.Cu" signal)
 		(31 "B.Cu" signal)
-		(32 "B.Adhes" user "B.Adhesive")
-		(33 "F.Adhes" user "F.Adhesive")
 		(34 "B.Paste" user)
 		(35 "F.Paste" user)
@@
 		(38 "B.Mask" user)
 		(39 "F.Mask" user)
-		(40 "Dwgs.User" user "User.Drawings")
-		(41 "Cmts.User" user "User.Comments")
-		(42 "Eco1.User" user "User.Eco1")
-		(43 "Eco2.User" user "User.Eco2")
 		(44 "Edge.Cuts" user)
 		(45 "Margin" user)
@@
 		(48 "B.Fab" user)
 		(49 "F.Fab" user)
-		(50 "User.1" user)
-		(51 "User.2" user)
-		(52 "User.3" user)
-		(53 "User.4" user)
-		(54 "User.5" user)
-		(55 "User.6" user)
-		(56 "User.7" user)
-		(57 "User.8" user)
-		(58 "User.9" user)
 	)
 	(setup
@@
 	(net 6 "unconnected-(U1-D2-Pad13)")
 	(net 7 "unconnected-(U1-Tx-Pad16)")
-	(net 8 "unconnected-(U1-GND-Pad10)")
+	(net 8 "GND")
 	(net 9 "unconnected-(U1-D3-Pad12)")
 	(net 10 "unconnected-(U1-D6-Pad5)")
@@
 	(net 17 "unconnected-(U2-1A-Pad2)")
 	(net 18 "unconnected-(U2-EN3,4-Pad9)")
-	(net 19 "unconnected-(U2-GND-Pad12)")
-	(net 20 "unconnected-(U2-EN1,2-Pad1)")
-	(net 21 "unconnected-(U2-VCC2-Pad8)")
-	(net 22 "unconnected-(U2-2Y-Pad6)")
-	(net 23 "unconnected-(U2-4Y-Pad14)")
-	(net 24 "unconnected-(U2-4A-Pad15)")
-	(net 25 "unconnected-(U2-GND-Pad5)")
-	(net 26 "unconnected-(U2-2A-Pad7)")
-	(net 27 "unconnected-(U2-3Y-Pad11)")
-	(net 28 "unconnected-(U2-3A-Pad10)")
-	(net 29 "unconnected-(U2-1Y-Pad3)")
-	(net 30 "unconnected-(U2-VCC1-Pad16)")
-	(net 31 "unconnected-(U2-GND-Pad13)")
-	(net 32 "unconnected-(U2-GND-Pad4)")
+	(net 19 "unconnected-(U2-EN1,2-Pad1)")
+	(net 20 "unconnected-(U2-VCC2-Pad8)")
+	(net 21 "unconnected-(U2-2Y-Pad6)")
+	(net 22 "unconnected-(U2-4Y-Pad14)")
+	(net 23 "unconnected-(U2-4A-Pad15)")
+	(net 24 "unconnected-(U2-2A-Pad7)")
+	(net 25 "unconnected-(U2-3Y-Pad11)")
+	(net 26 "unconnected-(U2-3A-Pad10)")
+	(net 27 "unconnected-(U2-1Y-Pad3)")
+	(net 28 "unconnected-(U2-VCC1-Pad16)")
 	(footprint "Package_DIP:DIP-16_W7.62mm"
 		(layer "F.Cu")
-		(at 134.62 76.2)
+		(at 115.58 77.485)
 		(descr "16-lead though-hole mounted DIP package, row spacing 7.62 mm (300 mils)")
 		(tags "THT DIP DIL PDIP 2.54mm 7.62mm 300mil")
@@
 			(layers "*.Cu" "*.Mask")
 			(remove_unused_layers no)
-			(net 20 "unconnected-(U2-EN1,2-Pad1)")
+			(net 19 "unconnected-(U2-EN1,2-Pad1)")
 			(pinfunction "EN1,2")
 			(pintype "input")
@@
 			(layers "*.Cu" "*.Mask")
 			(remove_unused_layers no)
-			(net 29 "unconnected-(U2-1Y-Pad3)")
+			(net 27 "unconnected-(U2-1Y-Pad3)")
 			(pinfunction "1Y")
 			(pintype "output")
@@
 			(layers "*.Cu" "*.Mask")
 			(remove_unused_layers no)
-			(net 32 "unconnected-(U2-GND-Pad4)")
+			(net 8 "GND")
 			(pinfunction "GND")
 			(pintype "power_in")
@@
 			(layers "*.Cu" "*.Mask")
 			(remove_unused_layers no)
-			(net 25 "unconnected-(U2-GND-Pad5)")
+			(net 8 "GND")
 			(pinfunction "GND")
 			(pintype "power_in")
@@
 			(layers "*.Cu" "*.Mask")
 			(remove_unused_layers no)
-			(net 22 "unconnected-(U2-2Y-Pad6)")
+			(net 21 "unconnected-(U2-2Y-Pad6)")
 			(pinfunction "2Y")
 			(pintype "output")
@@
 			(layers "*.Cu" "*.Mask")
 			(remove_unused_layers no)
-			(net 26 "unconnected-(U2-2A-Pad7)")
+			(net 24 "unconnected-(U2-2A-Pad7)")
 			(pinfunction "2A")
 			(pintype "input")
@@
 			(layers "*.Cu" "*.Mask")
 			(remove_unused_layers no)
-			(net 21 "unconnected-(U2-VCC2-Pad8)")
+			(net 20 "unconnected-(U2-VCC2-Pad8)")
 			(pinfunction "VCC2")
 			(pintype "power_in")
@@
 			(layers "*.Cu" "*.Mask")
 			(remove_unused_layers no)
-			(net 28 "unconnected-(U2-3A-Pad10)")
+			(net 26 "unconnected-(U2-3A-Pad10)")
 			(pinfunction "3A")
 			(pintype "input")
@@
 			(layers "*.Cu" "*.Mask")
 			(remove_unused_layers no)
-			(net 27 "unconnected-(U2-3Y-Pad11)")
+			(net 25 "unconnected-(U2-3Y-Pad11)")
 			(pinfunction "3Y")
 			(pintype "output")
@@
 			(layers "*.Cu" "*.Mask")
 			(remove_unused_layers no)
-			(net 19 "unconnected-(U2-GND-Pad12)")
+			(net 8 "GND")
 			(pinfunction "GND")
 			(pintype "power_in")
@@
 			(layers "*.Cu" "*.Mask")
 			(remove_unused_layers no)
-			(net 31 "unconnected-(U2-GND-Pad13)")
+			(net 8 "GND")
 			(pinfunction "GND")
 			(pintype "power_in")
@@
 			(layers "*.Cu" "*.Mask")
 			(remove_unused_layers no)
-			(net 23 "unconnected-(U2-4Y-Pad14)")
+			(net 22 "unconnected-(U2-4Y-Pad14)")
 			(pinfunction "4Y")
 			(pintype "output")
@@
 			(layers "*.Cu" "*.Mask")
 			(remove_unused_layers no)
-			(net 24 "unconnected-(U2-4A-Pad15)")
+			(net 23 "unconnected-(U2-4A-Pad15)")
 			(pinfunction "4A")
 			(pintype "input")
@@
 			(layers "*.Cu" "*.Mask")
 			(remove_unused_layers no)
-			(net 30 "unconnected-(U2-VCC1-Pad16)")
+			(net 28 "unconnected-(U2-VCC1-Pad16)")
 			(pinfunction "VCC1")
 			(pintype "power_in")
@@
 			(layers "*.Cu" "*.Mask")
 			(remove_unused_layers no)
-			(net 8 "unconnected-(U1-GND-Pad10)")
+			(net 8 "GND")
 			(pinfunction "GND")
 			(pintype "power_in")

Commit message: Continued the KeyCAD for the circuit board
Parts:
- added C1: C_Polarized, Capacitor_THT:C_Radial_D8.0mm_H11.5mm_P3.50mm, F.Cu at (174.6, 83.8)
- added J1: Conn_01x02_Pin, Connector_PinSocket_2.54mm:PinSocket_1x02_P2.54mm_Vertical, F.Cu at (137.8, 80.0)
- added J2: Conn_01x02_Pin, Connector_PinSocket_2.54mm:PinSocket_1x02_P2.54mm_Vertical, F.Cu at (137.8, 69.9)
- added J3: battery, project:battery wires, F.Cu at (172.7, 92.1)
- added J6: Conn_01x04_Pin, Connector_JST:JST_SH_SM04B-SRSS-TB_1x04-1MP_P1.00mm_Horizontal, B.Cu at (144.8, 94.2)
- added J7: Conn_01x06_Pin, Connector_PinHeader_2.54mm:PinHeader_2x03_P2.54mm_Vertical, F.Cu at (171.4, 69.2)
- added R1: R, Resistor_THT:R_Axial_DIN0204_L3.6mm_D1.6mm_P5.08mm_Horizontal, F.Cu at (165.1, 96.5)
- added R2: R, Resistor_THT:R_Axial_DIN0204_L3.6mm_D1.6mm_P5.08mm_Horizontal, F.Cu at (156.2, 95.2)
- added REF**: MountingHole_2.2mm_M2_DIN965_Pad_TopBottom, MountingHole:MountingHole_2.2mm_M2_DIN965_Pad_TopBottom, F.Cu at (137.8, 88.3)
- added REF**: MountingHole_2.2mm_M2_DIN965_Pad_TopBottom, MountingHole:MountingHole_2.2mm_M2_DIN965_Pad_TopBottom, F.Cu at (137.8, 64.1)
- added REF**: MountingHole_2.2mm_M2_DIN965_Pad_TopBottom, MountingHole:MountingHole_2.2mm_M2_DIN965_Pad_TopBottom, F.Cu at (172.7, 64.1)
- moved U2 47.6 mm to (161.3, 90.8), turned to 180 degrees
- moved U1 17.5 mm to (155.1, 79.7)
Connections:
- U1 pad 13: unconnected-(U1-D2-Pad13) -> Net-(J6-Pin_3)
- U1 pad 14: unconnected-(U1-D1-Pad14) -> Net-(J6-Pin_4)
- U1 pad 2: unconnected-(U1-A0-Pad2) -> Net-(U1-A0)
- U1 pad 3: unconnected-(U1-D0-Pad3) -> Net-(U1-D0)
- U1 pad 4: unconnected-(U1-D5-Pad4) -> Net-(U1-D5)
- U1 pad 5: unconnected-(U1-D6-Pad5) -> Net-(U1-D6)
- U1 pad 6: unconnected-(U1-D7-Pad6) -> Net-(U1-D7)
- U1 pad 8: unconnected-(U1-3.3V-Pad8) -> +3.3V
- U1 pad 9: unconnected-(U1-5V-Pad9) -> Net-(J3-Pin_1)
- U2 pad 1: unconnected-(U2-EN1,2-Pad1) -> +3.3V
- U2 pad 10: unconnected-(U2-3A-Pad10) -> Net-(U1-D5)
- U2 pad 11: unconnected-(U2-3Y-Pad11) -> Net-(J1-Pin_2)
- U2 pad 14: unconnected-(U2-4Y-Pad14) -> Net-(J1-Pin_1)
- U2 pad 15: unconnected-(U2-4A-Pad15) -> Net-(U1-D6)
- U2 pad 16: unconnected-(U2-VCC1-Pad16) -> Net-(J3-Pin_1)
- U2 pad 2: unconnected-(U2-1A-Pad2) -> Net-(U1-D7)
- U2 pad 3: unconnected-(U2-1Y-Pad3) -> Net-(J2-Pin_2)
- U2 pad 6: unconnected-(U2-2Y-Pad6) -> Net-(J2-Pin_1)
- U2 pad 7: unconnected-(U2-2A-Pad7) -> Net-(U1-D0)
- U2 pad 8: unconnected-(U2-VCC2-Pad8) -> Net-(J3-Pin_1)
- U2 pad 9: unconnected-(U2-EN3,4-Pad9) -> +3.3V
Routing:
- net Net-(J3-Pin_1): track 0.00 -> 52.4 mm
- added copper zone on F.Cu, net GND
Other:
- board size 66 x 63.5 mm -> 43.8 x 40 mm

Commit message: finished the KiCAD and created Gerbers
Parts:
- added G***: LOGO, LOGO, F.Cu at (169.5, 61.6)
- added G***: LOGO, LOGO, B.Cu at (152.4, 95.2)
- moved REF** 1.91 mm to (174.6, 64.1)
Routing:
- net Net-(J6-Pin_3): track 0.00 -> 60.3 mm
- net Net-(U1-A0): track 0.00 -> 58.8 mm
- net +3.3V: track 0.00 -> 48.1 mm
- net Net-(J6-Pin_4): track 0.00 -> 47.2 mm
- net Net-(J2-Pin_2): track 0.00 -> 37.4 mm
- net Net-(J1-Pin_1): track 0.00 -> 35.0 mm
- net Net-(J2-Pin_1): track 0.00 -> 30.7 mm
- net Net-(J1-Pin_2): track 0.00 -> 27.2 mm
- net Net-(J3-Pin_1): track 52.4 -> 77.5 mm
- net Net-(U1-D7): track 0.00 -> 19.6 mm, vias 0 -> 2
- net Net-(U1-D0): track 0.00 -> 18.8 mm, vias 0 -> 2
- net (no net): track 0.00 -> 16.1 mm
- net Net-(U1-D6): track 0.00 -> 13.0 mm
- net Net-(U1-D5): track 0.00 -> 11.2 mm, vias 0 -> 2
- net GND: track 0.00 -> 2.54 mm, vias 0 -> 1
Other:
- board size 43.8 x 40 mm -> 44.4 x 40 mm
- board text added: "#1"
- board text added: "#2"
- board text added: "#A"
- board text added: "#B"
- board text added: "+"
- board text added: "-"
- board text added: "BAT"
- board text added: "GND"
- board text added: "GPIO"
- board text added: "RCM D1 V 1.0"
- board text added: "https://github.com/rcmgames/RCM-Hardware-D1"
